File: MyPad PCB Files/MyPad.kicad_pcb (KiCad board)
At the start: 2 copper layers, 67 x 103 mm, 21 parts, among them J1 Conn_01x04_Pin, SW1 SW_Push, SW10 RotaryEncoder_Switch, SW2 SW_Push, SW3 SW_Push, SW4 SW_Push, SW5 SW_Push, SW6 SW_Push, SW7 SW_Push, SW8 SW_Push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

Commit message: Add files via upload
Other:
- board size 67 x 103 mm -> 67 x 102 mm
Changed lines of the file:
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@@
 	)
 	(footprint "Button_Switch_Keyboard:SW_Cherry_MX_1.00u_PCB"
+		(locked yes)
 		(layer "F.Cu")
 		(at 121.54 99.23)
@@
 	(gr_rect
 		(start 106 56)
-		(end 173 159)
+		(end 173 158)
 		(stroke
 			(width 0.05)
@@
 	)
 	(gr_circle
-		(center 169.5 155)
-		(end 172 155)
+		(center 169.5 152.5)
+		(end 172 152.5)
 		(stroke
 			(width 0.05)
@@
 	)
 	(gr_circle
-		(center 110 155)
-		(end 112.5 155)
+		(center 110 152.5)
+		(end 112.5 152.5)
 		(stroke
 			(width 0.05)
@@
 	)
 	(gr_text "MyPad\nMade by Isaac Lau\n(17, Hong Kong)"
-		(at 108.5 150.5 0)
+		(at 108.5 148.5 0)
 		(layer "F.Cu")
 		(effects

Commit message: Add files via upload
Routing:
- net Net-(U1-P2_D8_SCK): track 119.8 -> 247.2 mm
- net Net-(U1-P4_D9_MISO): track 142.5 -> 242.0 mm
- net Net-(U1-P3_D10_MOSI): track 111.5 -> 130.0 mm
- net GND: track 176.7 -> 168.4 mm
- net Column 0: track 82.3 -> 84.6 mm
Other:
- board size 67 x 102 mm -> 67 x 99.5 mm
